File: lcd-mall-LMT040WV004C/mipi-dsi-in.kicad_sch (KiCad schematic)
At the start: 1 part, among them J1 1-1734248-5

Commit message: Fix parts for board LMT040WM004C
Parts:
- J1: LCSC (none) -> C2922285
Changed lines of the file:
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@@
+			)
+		)
+		(property "LCSC" "C2922285"
+			(at 110.49 110.49 0)
+			(effects
+				(font
+					(size 1.27 1.27)
+				)
+				(hide yes)
 			)
 		)
