File: lcd-mall-LMT040WV004C/mipi-dsi-out.kicad_sch (KiCad schematic)
At the start: 8 parts, among them J2 FFC2B35-24-G, SW1 SMD-BUTTON_4P-5.2X5.2X1.5MM-S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

Commit message: Fix names, footprints, and silkscreen of the pcb's
Parts:
- SW1: footprint custom:SW4-SMD-5.2X5.2X1.5MM -> SMD-BUTTON_4P-5.2X5.2X1.5MM-SKQGADE010_:SW4-SMD-5.2X5.2X1.5MM
Changed lines of the file:
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@@
 			)
 		)
-		(property "Footprint" "custom:SW4-SMD-5.2X5.2X1.5MM"
+		(property "Footprint" "SMD-BUTTON_4P-5.2X5.2X1.5MM-SKQGADE010_:SW4-SMD-5.2X5.2X1.5MM"
 			(at 246.38 45.72 0)
 			(effects

Commit message: Fix parts for board LMT040WM004C
Parts:
- removed C8: 10nF, Capacitor_SMD:C_0603_1608Metric, symbol Device:C
- removed J2: FFC2B35-24-G, FFC2B3524G, symbol FFC2B35-24-G:FFC2B35-24-G
- added FPC1: 0.5K-QX-24PWB, easyeda2kicad:FPC-SMD_24P-P0.50_HDGC_0.5K-QX-24PWB, symbol easyeda2kicad:0.5K-QX-24PWB
- C4: LCSC C5189821 -> C126631
Connections:
- net +1V8: now also FPC1.16, FPC1.17
- net +3V3: now also FPC1.19, FPC1.20
- net CLK_C_N: now also FPC1.8
- net CLK_C_P: now also FPC1.7
- net D0_N: now also FPC1.2
- net D0_P: now also FPC1.1
- net D1_N: now also FPC1.5
- net D1_P: now also FPC1.4
- net GND: now also FPC1.12, FPC1.15, FPC1.3, FPC1.6, FPC1.9
- net LEDA: now also FPC1.24
- net LEDK: now also FPC1.22
- net RST: now also FPC1.18
- net at TP1.1: now also FPC1.21
Changed lines of the file:
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@@
-	)
-	(junction
-		(at 243.84 110.49)
-		(diameter 0)
-		(color 0 0 0 0)
 	)
 	(junction
@@
 	)
 	(junction
-		(at 243.84 118.11)
-		(diameter 0)
-		(color 0 0 0 0)
-	)
-	(junction
 		(at 101.6 96.52)
 		(diameter 0)
@@
 	)
 	(no_connect
+		(at 111.76 53.34)
+	)
+	(no_connect
 		(at 104.14 91.44)
-	)
-	(no_connect
-		(at 129.54 58.42)
 	)
 	(no_connect
@@
 	)
 	(no_connect
-		(at 129.54 60.96)
+		(at 111.76 121.92)
 	)
 	(no_connect
@@
 		)
 	)
-	(wire
-		(pts
-			(xy 243.84 110.49) (xy 256.54 110.49)
-		)
-		(stroke
-			(width 0)
-			(type default)
-		)
-	)
 	(polyline
 		(pts
@@
 	(wire
 		(pts
-			(xy 231.14 110.49) (xy 243.84 110.49)
+			(xy 231.14 110.49) (xy 256.54 110.49)
 		)
 		(stroke
@@
 	(wire
 		(pts
-			(xy 243.84 118.11) (xy 256.54 118.11)
+			(xy 231.14 118.11) (xy 256.54 118.11)
 		)
 		(stroke
@@
 			(width 0)
 			(type dash)
-		)
-	)
-	(wire
-		(pts
-			(xy 231.14 118.11) (xy 243.84 118.11)
-		)
-		(stroke
-			(width 0)
-			(type default)
 		)
 	)
@@
 	(symbol
 		(lib_id "Device:C")
-		(at 243.84 114.3 0)
-		(unit 1)
-		(exclude_from_sim no)
-		(in_bom yes)
-		(on_board yes)
-		(dnp no)
-		(fields_autoplaced yes)
-		(property "Reference" "C8"
-			(at 247.65 113.0299 0)
-			(effects
-				(font
-					(size 1.27 1.27)
-				)
-				(justify left)
-			)
-		)
-		(property "Value" "10nF"
-			(at 247.65 115.5699 0)
-			(effects
-				(font
-					(size 1.27 1.27)
-				)
-				(justify left)
-			)
-		)
-		(property "Footprint" "Capacitor_SMD:C_0603_1608Metric"
-			(at 244.8052 118.11 0)
-			(effects
-				(font
-					(size 1.27 1.27)
-				)
-				(hide yes)
-			)
-		)
-		(property "Datasheet" "~"
-			(at 243.84 114.3 0)
-			(effects
-				(font
-					(size 1.27 1.27)
-				)
-				(hide yes)
-			)
-		)
-		(property "Description" "Unpolarized capacitor"
-			(at 243.84 114.3 0)
-			(effects
-				(font
-					(size 1.27 1.27)
-				)
-				(hide yes)
-			)
-		)
-		(property "LCSC" "C525264"
-			(at 243.84 114.3 0)
-			(effects
-				(font
-					(size 1.27 1.27)
-				)
-				(hide yes)
-			)
-		)
-		(pin "1"
-		)
-		(pin "2"
-		)
-		(instances
-			(project "50-24-fpc-adapter-board"
-				(path "/32028fb8-27d2-4a38-96f3-0c731f94a0fb/ea03a3c5-5ac0-4618-bb08-06acbdff3056"
-					(reference "C8")
-					(unit 1)
-				)
-			)
-		)
-	)
-	(symbol
-		(lib_id "Device:C")
 		(at 256.54 114.3 0)
 		(unit 1)
@@
 				(path "/32028fb8-27d2-4a38-96f3-0c731f94a0fb/ea03a3c5-5ac0-4618-bb08-06acbdff3056"
 					(reference "#PWR08")
+					(unit 1)
+				)
+			)
+		)
+	)
+	(symbol
+		(lib_id "easyeda2kicad:0.5K-QX-24PWB")
+		(at 107.95 87.63 0)
+		(unit 1)
+		(exclude_from_sim no)
+		(in_bom yes)
+		(on_board yes)
+		(dnp no)
+		(fields_autoplaced yes)
+		(property "Reference" "FPC1"
+			(at 114.3 86.3599 0)
+			(effects
+				(font
+					(size 1.27 1.27)
+				)
+				(justify left)
+			)
+		)
+		(property "Value" "0.5K-QX-24PWB"
+			(at 114.3 88.8999 0)
+			(effects
+				(font
+					(size 1.27 1.27)
+				)
+				(justify left)
+			)
+		)
+		(property "Footprint" "easyeda2kicad:FPC-SMD_24P-P0.50_HDGC_0.5K-QX-24PWB"
+			(at 107.95 129.54 0)
+			(effects
+				(font
+					(size 1.27 1.27)
+				)
+				(hide yes)
+			)
+		)
+		(property "Datasheet" ""
+			(at 107.95 87.63 0)
+			(effects
+				(font
+					(size 1.27 1.27)
+				)
+				(hide yes)
+			)
+		)
+		(property "Description" ""
+			(at 107.95 87.63 0)
+			(effects
+				(font
+					(size 1.27 1.27)
+				)
+				(hide yes)
+			)
+		)
+		(property "LCSC Part" "C2919484"
+			(at 107.95 132.08 0)
+			(effects
+				(font
+					(size 1.27 1.27)
+				)
+				(hide yes)
+			)
+		)
+		(pin "6"
+		)
+		(pin "9"
+		)
+		(pin "19"
+		)
+		(pin "7"
+		)
+		(pin "24"
+		)
+		(pin "14"
+		)
+		(pin "11"
+		)
+		(pin "1"
+		)
+		(pin "10"
+		)
+		(pin "25"
+		)
+		(pin "17"
+		)
+		(pin "18"
+		)
+		(pin "23"
+		)
+		(pin "15"
+		)
+		(pin "12"
+		)
+		(pin "13"
+		)
+		(pin "2"
+		)
+		(pin "5"
+		)
+		(pin "16"
+		)
+		(pin "26"
+		)
+		(pin "20"
+		)
+		(pin "22"
+		)
+		(pin "4"
+		)
+		(pin "21"
+		)
+		(pin "3"
+		)
+		(pin "8"
+		)
+		(instances
+			(project "50-24-fpc-adapter-board"
+				(path "/32028fb8-27d2-4a38-96f3-0c731f94a0fb/ea03a3c5-5ac0-4618-bb08-06acbdff3056"
+					(reference "FPC1")
 					(unit 1)
 				)
@@
 	)
 	(symbol
-		(lib_id "FFC2B35-24-G:FFC2B35-24-G")
-		(at 129.54 58.42 0)
-		(mirror y)
-		(unit 1)
-		(exclude_from_sim no)
-		(in_bom yes)
-		(on_board yes)
-		(dnp no)
-		(property "Reference" "J2"
-			(at 116.84 50.8 0)
-			(effects
-				(font
-					(size 1.27 1.27)
-				)
-			)
-		)
-		(property "Value" "FFC2B35-24-G"
-			(at 116.84 53.34 0)
-			(effects
-				(font
-					(size 1.27 1.27)
-				)
-			)
-		)
-		(property "Footprint" "FFC2B3524G"
-			(at 107.95 153.34 0)
-			(effects
-				(font
-					(size 1.27 1.27)
-				)
-				(justify left top)
-				(hide yes)
-			)
-		)
-		(property "Datasheet" "https://gct.co/connector/ffc2b35"
-			(at 107.95 253.34 0)
-			(effects
-				(font
-					(size 1.27 1.27)
-				)
-				(justify left top)
-				(hide yes)
-			)
-		)
-		(property "Description" "GCT (GLOBAL CONNECTOR TECHNOLOGY) - FFC2B35-24-G - FFC / FPC Board Connector, 0.5 mm, 24 Contacts, Receptacle, FFC2B35 Series"
-			(at 129.54 58.42 0)
-			(effects
-				(font
-					(size 1.27 1.27)
-				)
-				(hide yes)
-			)
-		)
-		(property "Height" "2.2"
-			(at 107.95 453.34 0)
-			(effects
-				(font
-					(size 1.27 1.27)
-				)
-				(justify left top)
-				(hide yes)
-			)
-		)
-		(property "Mouser Part Number" "640-FFC2B35-24-G"
-			(at 107.95 553.34 0)
-			(effects
-				(font
-					(size 1.27 1.27)
-				)
-				(justify left top)
-				(hide yes)
-			)
-		)
-		(property "Mouser Price/Stock" "https://www.mouser.co.uk/ProductDetail/GCT/FFC2B35-24-G?qs=Li%252BoUPsLEnvPfOHuwRN%252BFA%3D%3D"
-			(at 107.95 653.34 0)
-			(effects
-				(font
-					(size 1.27 1.27)
-				)
-				(justify left top)
-				(hide yes)
-			)
-		)
-		(property "Manufacturer_Name" "GCT (GLOBAL CONNECTOR TECHNOLOGY)"
-			(at 107.95 753.34 0)
-			(effects
-				(font
-					(size 1.27 1.27)
-				)
-				(justify left top)
-				(hide yes)
-			)
-		)
-		(property "Manufacturer_Part_Number" "FFC2B35-24-G"
-			(at 107.95 853.34 0)
-			(effects
-				(font
-					(size 1.27 1.27)
-				)
-				(justify left top)
-				(hide yes)
-			)
-		)
-		(pin "2"
-		)
-		(pin "21"
-		)
-		(pin "5"
-		)
-		(pin "19"
-		)
-		(pin "24"
-		)
-		(pin "23"
-		)
-		(pin "8"
-		)
-		(pin "18"
-		)
-		(pin "20"
-		)
-		(pin "MP2"
-		)
-		(pin "9"
-		)
-		(pin "1"
-		)
-		(pin "17"
-		)
-		(pin "7"
-		)
-		(pin "4"
-		)
-		(pin "6"
-		)
-		(pin "3"
-		)
-		(pin "15"
-		)
-		(pin "MP1"
-		)
-		(pin "10"
-		)
-		(pin "14"
-		)
-		(pin "12"
-		)
-		(pin "13"
-		)
-		(pin "22"
-		)
-		(pin "16"
-		)
-		(pin "11"
-		)
-		(instances
-			(project "50-24-fpc-adapter-board"
-				(path "/32028fb8-27d2-4a38-96f3-0c731f94a0fb/ea03a3c5-5ac0-4618-bb08-06acbdff3056"
-					(reference "J2")
-					(unit 1)
-				)
-			)
-		)
-	)
-	(symbol
 		(lib_id "Device:C")
 		(at 227.33 46.99 0)
@@
 			)
 		)
-		(property "LCSC" "C5189821"
+		(property "LCSC" "C126631"
 			(at 227.33 46.99 0)
 			(effects

Commit message: Fixed lmt040wv004c board for production @ JLCPCB
Parts:
- FPC1: LCSC (none) -> C2919484; LCSC Part C2919484 -> (none)
Changed lines of the file:
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@@
 			)
 		)
-		(property "LCSC Part" "C2919484"
+		(property "LCSC" "C2919484"
 			(at 107.95 132.08 0)
 			(effects
